Commit message: Update 06-flexible.urdf

File: 06-flexible.urdf (robot description, URDF)
Before this commit: robot visual, 16 links, 15 joints
Links:
- link left_gripper: geometry visual mesh filename=package://manipulator/meshes/l_finger.dae
- link left_tip: geometry visual mesh filename=package://manipulator/meshes/l_finger_tip.dae
- link right_gripper: geometry visual mesh filename=package://manipulator/meshes/l_finger.dae
- link right_tip: geometry visual mesh filename=package://manipulator/meshes/l_finger_tip.dae
